Commit message: 增加了URDF文件引入

File: src/robot/urdf/robot.urdf (robot description, URDF)
Before this commit: robot robot, 9 links, 8 joints
Links:
- removed link base_footprint
- removed link controller_Link
- removed link idar_Link
- removed link imu_Link
- removed link wheel_1_Link
- removed link wheel_2_Link
- removed link wheel_3_Link
- removed link wheel_4_Link
- added link livox_frame, mass 0.190304028239138; collision mesh filename=package://robot/meshes/livox_frame.STL; visual mesh filename=package://robot/meshes/livox_frame.STL
- link base_link: mass 0.739736885196848 -> 2.34291090302096
Joints:
- removed joint base_footprint_joint
- removed joint controller_joint
- removed joint idar_joint
- removed joint imu_joint
- removed joint wheel_1_joint
- removed joint wheel_2_joint
- removed joint wheel_3_joint
- removed joint wheel_4_joint
- added joint livox_frame: type fixed, parent base_link, child livox_frame, origin xyz=0.0200000000000045 -0.0949999999999872 0.3228 rpy=0 0 0, axis 0 0 0
